File: robot_vr.brd (EAGLE design)
At the start: 160 x 100 mm, 34 parts, among them CN10 SSM-119-L-DV, CN7 SSM-119-L-DV

Commit message: Add files via upload
Routing:
- net GND: track 434.6 -> 449.1 mm
- net N$1: track 140.6 -> 149.5 mm
- net MOT-: track 309.4 -> 311.0 mm
Changed lines of the file:
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@@
 <?xml version="1.0" encoding="utf-8"?>
 <!DOCTYPE eagle SYSTEM "eagle.dtd">
-<eagle version="7.1.0">
+<eagle version="7.6.0">
 <drawing>
 <settings>
@@
 <wire x1="5.9436" y1="53.0352" x2="8.4582" y2="53.0352" width="0.254" layer="1"/>
 <wire x1="26.5176" y1="35.433" x2="26.67" y2="35.2275" width="0.254" layer="1"/>
-<wire x1="7.3152" y1="66.0654" x2="7.3152" y2="72.2376" width="0.254" layer="1"/>
-<wire x1="7.3152" y1="61.0362" x2="7.3152" y2="66.0654" width="0.254" layer="16"/>
-<wire x1="7.3152" y1="59.8932" x2="7.3152" y2="61.0362" width="0.254" layer="1"/>
+<wire x1="7.3152" y1="68.0974" x2="7.3152" y2="72.2376" width="0.254" layer="1"/>
+<wire x1="10.6172" y1="55.9562" x2="10.668" y2="55.9562" width="0.254" layer="16"/>
+<wire x1="10.668" y1="55.9562" x2="10.668" y2="68.072" width="0.254" layer="16"/>
+<wire x1="10.668" y1="68.072" x2="7.3152" y2="68.0974" width="0.254" layer="16"/>
+<wire x1="7.3152" y1="59.8932" x2="7.366" y2="56.134" width="0.254" layer="1"/>
+<wire x1="7.366" y1="56.134" x2="7.366" y2="55.9562" width="0.254" layer="1"/>
+<wire x1="7.366" y1="55.9562" x2="10.6172" y2="55.9562" width="0.254" layer="1"/>
 <wire x1="7.3152" y1="72.2376" x2="7.2875" y2="72.39" width="0.254" layer="1"/>
 <wire x1="7.3152" y1="59.8932" x2="7.2875" y2="59.69" width="0.254" layer="1"/>
@@
 <wire x1="35.8902" y1="13.9446" x2="35.6616" y2="13.716" width="0.254" layer="1"/>
 <wire x1="35.8902" y1="13.9446" x2="35.9825" y2="13.99" width="0.254" layer="1"/>
-<via x="7.3152" y="66.0654" extent="1-16" drill="0.6096"/>
-<via x="7.3152" y="61.0362" extent="1-16" drill="0.6096"/>
+<via x="7.3152" y="68.0974" extent="1-16" drill="0.6096"/>
+<via x="10.6172" y="55.9562" extent="1-16" drill="0.6096"/>
 <polygon width="0.4064" layer="1" isolate="0.4064" orphans="yes">
 <vertex x="160.274" y="100.076"/>
@@
 <wire x1="6.4008" y1="21.717" x2="6.35" y2="21.59" width="0.254" layer="1"/>
 <wire x1="7.0866" y1="64.6938" x2="7.2875" y2="64.77" width="0.254" layer="1"/>
-<wire x1="37.719" y1="28.575" x2="45.4735" y2="28.575" width="0.254" layer="1"/>
-<wire x1="21.4884" y1="28.575" x2="37.719" y2="28.575" width="0.254" layer="16"/>
+<wire x1="40.767" y1="28.575" x2="45.4735" y2="28.575" width="0.254" layer="1"/>
+<wire x1="21.4884" y1="28.575" x2="40.767" y2="28.575" width="0.254" layer="16"/>
 <wire x1="45.4914" y1="28.575" x2="45.4735" y2="28.575" width="0.254" layer="1"/>
 <via x="110.871" y="34.9758" extent="1-16" drill="0.6096"/>
 <via x="93.9546" y="34.9758" extent="1-16" drill="0.6096"/>
-<via x="37.719" y="28.575" extent="1-16" drill="0.6096"/>
+<via x="40.767" y="28.575" extent="1-16" drill="0.6096"/>
 <via x="21.4884" y="28.575" extent="1-16" drill="0.6096"/>
 <wire x1="84.2385" y1="29.33" x2="87.5722" y2="29.33" width="0.4064" layer="1"/>
@@
 <wire x1="30.48" y1="8.66" x2="30.734" y2="8.66" width="0.4064" layer="1"/>
 <wire x1="30.734" y1="8.66" x2="30.734" y2="3.81" width="0.4064" layer="1"/>
-<wire x1="34.5186" y1="27.6606" x2="35.8902" y2="29.0322" width="0.254" layer="1"/>
-<wire x1="27.8892" y1="27.6606" x2="34.5186" y2="27.6606" width="0.254" layer="16"/>
+<wire x1="39.0906" y1="27.4066" x2="35.8902" y2="29.0322" width="0.254" layer="1"/>
+<wire x1="27.8892" y1="27.6606" x2="39.0906" y2="27.4066" width="0.254" layer="16"/>
 <wire x1="3.8862" y1="3.6576" x2="27.8892" y2="27.6606" width="0.254" layer="16"/>
 <wire x1="35.8902" y1="29.0322" x2="35.9825" y2="29.23" width="0.254" layer="1"/>
 <wire x1="3.8862" y1="3.6576" x2="3.81" y2="3.81" width="0.254" layer="16"/>
 <wire x1="69.9516" y1="27.6606" x2="71.3232" y2="29.0322" width="0.254" layer="1"/>
-<wire x1="34.5186" y1="27.6606" x2="69.9516" y2="27.6606" width="0.254" layer="16"/>
+<wire x1="39.0906" y1="27.4066" x2="69.9516" y2="27.6606" width="0.254" layer="16"/>
 <wire x1="71.3232" y1="29.0322" x2="71.4765" y2="29.216" width="0.254" layer="1"/>
 <wire x1="104.4702" y1="29.0322" x2="106.7562" y2="29.0322" width="0.254" layer="1"/>
@@
 <wire x1="104.4702" y1="29.0322" x2="104.6988" y2="29.2608" width="0.254" layer="16"/>
 <wire x1="142.4178" y1="29.2608" x2="142.5185" y2="29.368" width="0.254" layer="1"/>
-<via x="34.5186" y="27.6606" extent="1-16" drill="0.6096"/>
+<via x="39.0906" y="27.4066" extent="1-16" drill="0.6096"/>
 <via x="69.9516" y="27.6606" extent="1-16" drill="0.6096"/>
 <via x="104.4702" y="29.0322" extent="1-16" drill="0.6096"/>
@@
 <wire x1="21.717" y1="15.5448" x2="21.59" y2="15.5725" width="0.254" layer="1"/>
 <wire x1="89.8398" y1="15.5448" x2="92.583" y2="15.5448" width="0.254" layer="1"/>
-<wire x1="58.5216" y1="15.5448" x2="89.8398" y2="15.5448" width="0.254" layer="16"/>
-<wire x1="57.15" y1="15.5448" x2="58.5216" y2="15.5448" width="0.254" layer="1"/>
+<wire x1="56.9976" y1="7.6708" x2="89.8398" y2="15.5448" width="0.254" layer="16"/>
+<wire x1="57.15" y1="15.5448" x2="56.9976" y2="7.6708" width="0.254" layer="1"/>
 <wire x1="92.583" y1="15.5448" x2="92.71" y2="15.5725" width="0.254" layer="1"/>
 <wire x1="57.15" y1="15.5448" x2="57.15" y2="15.5725" width="0.254" layer="1"/>
@@
 <wire x1="128.2446" y1="12.573" x2="128.27" y2="12.3675" width="0.254" layer="1"/>
 <via x="89.8398" y="15.5448" extent="1-16" drill="0.6096"/>
-<via x="58.5216" y="15.5448" extent="1-16" drill="0.6096"/>
+<via x="56.9976" y="7.6708" extent="1-16" drill="0.6096"/>
 <via x="115.6716" y="12.573" extent="1-16" drill="0.6096"/>
 <wire x1="3.81" y1="6.35" x2="12.3675" y2="6.35" width="0.4064" layer="1"/>

Commit message: Add files via upload
Parts:
- moved CAM 134.5 mm to (261.8, 162.2)
- moved DRVMOT1_POW 117.0 mm to (255.9, 44.6), turned to 180 degrees
- moved DRVMOT1_COM 107.8 mm to (255.9, 57.3), turned to 180 degrees
- moved C1 105.9 mm to (239.6, 36.9)
- moved CAPTEUR1_COM 105.9 mm to (231.8, 68.6), turned to 0 degrees
- moved CAPTEUR1_POW 105.5 mm to (231.8, 44.6)
- moved MOT1 103.3 mm to (252.2, 28.9), turned to 0 degrees
- moved DRVMOT2_POW 83.7 mm to (186.2, 44.6), turned to 180 degrees
- moved CN10 83.6 mm to (162.9, 139.6)
- moved CN7 83.6 mm to (101.9, 139.6)
- moved STOP_SENSOR1 82.6 mm to (22.9, 169.0)
- moved DRVMOT2_COM 76.2 mm to (186.2, 57.3), turned to 180 degrees
- moved C2 74.5 mm to (171.6, 35.9)
- moved CAPTEUR2_COM 74.0 mm to (162.1, 68.6), turned to 0 degrees
- moved CAPTEUR2_POW 73.6 mm to (162.1, 44.6)
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Connections:
- net N$1 renamed MOT+
Routing:
- net SUPPLY_COM: track 410.2 -> 998.2 mm, vias 4 -> 5
- net GND: track 449.1 -> 960.4 mm, vias 2 -> 17
- net MOT+: track 149.5 -> 413.6 mm, vias 3 -> 4
- net MOT-: track 311.0 -> 484.3 mm, vias 4 -> 8
- net CS: track 42.5 -> 176.6 mm
- net MOTOR1_STEP: track 83.5 -> 215.0 mm, vias 0 -> 2
- net SCK/TX: track 103.7 -> 216.5 mm, vias 0 -> 2
- net CURRENT_SENSOR1: track 92.5 -> 201.5 mm, vias 0 -> 2
- net MOTOR1_READY: track 72.6 -> 179.8 mm
- net MOTOR1_DIR: track 86.8 -> 189.9 mm
- net MOTOR5_SERVO: track 160.9 -> 259.0 mm, vias 0 -> 2
- net CURRENT_SENSOR4: track 46.2 -> 140.9 mm, vias 0 -> 2
- net CURRENT_SENSOR2: track 44.3 -> 135.3 mm, vias 0 -> 2
- net MOSI: track 109.3 -> 198.1 mm, vias 0 -> 2
- net MOTOR4_STEP: track 101.8 -> 183.2 mm
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- removed copper zone on layer 1, net GND
Other:
- board size 160 x 100 mm -> 283 x 184 mm
