File: robot_vr.brd (EAGLE design)
At the start: 283 x 184 mm, 34 parts, among them CN10 SSM-119-L-DV, CN7 SSM-119-L-DV

Commit message: Add files via upload
Connections:
- net CS: now also CAM.05; no longer CAM.04
- net MOSI: now also CAM.02; no longer CAM.01
- net SCK/TX: now also CAM.01; no longer CAM.02
- net SCL: now also CAM.04; no longer CAM.05
Routing:
- net SUPPLY_COM: track 998.2 -> 881.5 mm
- net CS: track 176.6 -> 112.7 mm
- net SCK/TX: track 216.5 -> 177.0 mm, vias 2 -> 0
- net SCL: track 99.9 -> 116.3 mm
- net MOSI: track 198.1 -> 202.1 mm, vias 2 -> 0
- net STOP_SENSOR4: track 112.0 -> 109.7 mm, vias 2 -> 0
- net STOP_SENSOR2: track 86.0 -> 83.7 mm, vias 2 -> 0
- net STOP_SENSOR3: track 89.5 -> 87.5 mm, vias 2 -> 0
- net STOP_SENSOR1: track 108.5 -> 106.6 mm, vias 2 -> 0
- net SDA/MISO/RX: track 162.9 -> 162.0 mm, vias 2 -> 0

Commit message: Add files via upload
Connections:
- net GND: now also CAPTEUR1_COM.01, CAPTEUR2_COM.01, CAPTEUR3_COM.01, CAPTEUR4_COM.01; no longer CAPTEUR1_COM.03, CAPTEUR2_COM.03, CAPTEUR3_COM.03, CAPTEUR4_COM.03
- net SUPPLY_COM: now also CAPTEUR1_COM.03, CAPTEUR2_COM.03, CAPTEUR3_COM.03, CAPTEUR4_COM.03; no longer CAPTEUR1_COM.01, CAPTEUR2_COM.01, CAPTEUR3_COM.01, CAPTEUR4_COM.01
Routing:
- net GND: track 960.4 -> 1022.8 mm, vias 17 -> 19
- net SUPPLY_COM: track 881.5 -> 891.6 mm
Changed lines of the file:
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@@
 <?xml version="1.0" encoding="utf-8"?>
 <!DOCTYPE eagle SYSTEM "eagle.dtd">
-<eagle version="9.6.2">
+<eagle version="7.6.0">
 <drawing>
 <settings>
 <setting alwaysvectorfont="no"/>
-<setting keepoldvectorfont="yes"/>
 <setting verticaltext="up"/>
 </settings>
@@
 <param name="dpMaxLengthDifference" value="10mm"/>
 <param name="dpGapFactor" value="2.5"/>
+<param name="checkGrid" value="0"/>
 <param name="checkAngle" value="0"/>
 <param name="checkFont" value="1"/>
 <param name="checkRestrict" value="1"/>
-<param name="checkStop" value="0"/>
-<param name="checkValues" value="0"/>
-<param name="checkNames" value="1"/>
-<param name="checkWireStubs" value="1"/>
-<param name="checkPolygonWidth" value="0"/>
 <param name="useDiameter" value="13"/>
 <param name="maxErrors" value="50"/>
@@
 <signals>
 <signal name="GND">
-<contactref element="CAPTEUR1_COM" pad="03"/>
-<contactref element="CAPTEUR2_COM" pad="03"/>
-<contactref element="CAPTEUR3_COM" pad="03"/>
-<contactref element="CAPTEUR4_COM" pad="03"/>
 <contactref element="DRVMOT1_POW" pad="08"/>
 <contactref element="DRVMOT2_POW" pad="08"/>
@@
 <wire x1="9.83" y1="70.1825" x2="10" y2="70.1825" width="0.3048" layer="16"/>
 <wire x1="10" y1="70.1825" x2="10" y2="91.47" width="0.3048" layer="16"/>
-<wire x1="34.12" y1="70.1825" x2="27" y2="70.1825" width="0.3048" layer="1"/>
-<wire x1="27" y1="70.1825" x2="9.83" y2="70.1825" width="0.3048" layer="1"/>
+<wire x1="27" y1="70.1825" x2="24" y2="70.1825" width="0.3048" layer="1"/>
+<wire x1="24" y1="70.1825" x2="9.83" y2="70.1825" width="0.3048" layer="1"/>
 <wire x1="9.83" y1="70.1825" x2="10" y2="70.1825" width="0.3048" layer="1"/>
 <wire x1="10" y1="70.1825" x2="10" y2="57" width="0.3048" layer="16"/>
@@
 <via x="27" y="70.1825" extent="1-16" drill="0.8" diameter="1.27"/>
 <via x="76" y="46.1825" extent="1-16" drill="0.8" diameter="1.27"/>
-<wire x1="92.36" y1="70.1825" x2="76" y2="70.1825" width="0.3048" layer="1"/>
 <wire x1="76" y1="70.1825" x2="76" y2="46.1825" width="0.3048" layer="16"/>
-<via x="76" y="70.1825" extent="1-16" drill="0.8" diameter="1.27"/>
 <wire x1="127.9" y1="46.1825" x2="131" y2="46.1825" width="0.3048" layer="1"/>
 <wire x1="131" y1="46.1825" x2="131" y2="23" width="0.3048" layer="16"/>
 <wire x1="131" y1="23" x2="76" y2="23" width="0.3048" layer="16"/>
 <via x="131" y="46.1825" extent="1-16" drill="0.8" diameter="1.27"/>
-<wire x1="159.6" y1="70.1825" x2="154" y2="70.1825" width="0.3048" layer="1"/>
-<wire x1="154" y1="70.1825" x2="154" y2="46" width="0.3048" layer="16"/>
-<wire x1="154" y1="46" x2="131" y2="46" width="0.3048" layer="16"/>
 <wire x1="131" y1="46" x2="131" y2="46.1825" width="0.3048" layer="1"/>
-<via x="154" y="70.1825" extent="1-16" drill="0.8" diameter="1.27"/>
 <wire x1="195.04" y1="46.1825" x2="198" y2="46.1825" width="0.3048" layer="1"/>
 <wire x1="198" y1="46.1825" x2="198" y2="46" width="0.3048" layer="1"/>
 <wire x1="198" y1="46" x2="198" y2="23" width="0.3048" layer="16"/>
 <wire x1="198" y1="23" x2="131" y2="23" width="0.3048" layer="16"/>
-<wire x1="229.26" y1="70.1825" x2="215" y2="70.1825" width="0.3048" layer="1"/>
-<wire x1="215" y1="70.1825" x2="215" y2="46" width="0.3048" layer="16"/>
 <wire x1="215" y1="46" x2="198" y2="46" width="0.3048" layer="16"/>
 <via x="198" y="46" extent="1-16" drill="0.8" diameter="1.27"/>
-<via x="215" y="70.1825" extent="1-16" drill="0.8" diameter="1.27"/>
 <wire x1="264.76" y1="46.1825" x2="269" y2="46.1825" width="0.3048" layer="1"/>
 <wire x1="269" y1="46.1825" x2="269" y2="23" width="0.3048" layer="16"/>
 <wire x1="269" y1="23" x2="198" y2="23" width="0.3048" layer="16"/>
 <via x="269" y="46.1825" extent="1-16" drill="0.8" diameter="1.27"/>
+<contactref element="CAPTEUR4_COM" pad="01"/>
+<contactref element="CAPTEUR3_COM" pad="01"/>
+<contactref element="CAPTEUR2_COM" pad="01"/>
+<contactref element="CAPTEUR1_COM" pad="01"/>
+<wire x1="39.2" y1="79" x2="24" y2="79" width="0.3048" layer="16"/>
+<wire x1="24" y1="79" x2="24" y2="70.1825" width="0.3048" layer="1"/>
+<wire x1="39.2" y1="79" x2="39.2" y2="70.1825" width="0.3048" layer="1"/>
+<via x="39.2" y="79" extent="1-16" drill="0.8" diameter="1.27"/>
+<via x="24" y="79" extent="1-16" drill="0.8" diameter="1.27"/>
+<wire x1="76" y1="70.1825" x2="89" y2="70.1825" width="0.3048" layer="16"/>
+<wire x1="89" y1="70.1825" x2="89" y2="73" width="0.3048" layer="16"/>
+<wire x1="89" y1="73" x2="97.44" y2="73" width="0.3048" layer="16"/>
+<wire x1="97.44" y1="73" x2="97.44" y2="70.1825" width="0.3048" layer="1"/>
+<via x="97.44" y="73" extent="1-16" drill="0.8" diameter="1.27"/>
+<wire x1="164.68" y1="70.1825" x2="168" y2="70.1825" width="0.3048" layer="1"/>
+<wire x1="168" y1="70.1825" x2="168" y2="50" width="0.3048" layer="16"/>
+<wire x1="168" y1="50" x2="131" y2="50" width="0.3048" layer="16"/>
+<wire x1="131" y1="50" x2="131" y2="46.1825" width="0.3048" layer="16"/>
+<via x="168" y="70.1825" extent="1-16" drill="0.8" diameter="1.27"/>
+<wire x1="234.34" y1="70.1825" x2="239" y2="70.1825" width="0.3048" layer="1"/>
+<wire x1="239" y1="70.1825" x2="239" y2="53" width="0.3048" layer="16"/>
+<wire x1="239" y1="53" x2="215" y2="53" width="0.3048" layer="16"/>
+<wire x1="215" y1="53" x2="215" y2="46" width="0.3048" layer="16"/>
+<via x="239" y="70.1825" extent="1-16" drill="0.8" diameter="1.27"/>
 </signal>
 <signal name="SCK/TX">
@@
 <contactref element="DRVMOT4_COM" pad="03"/>
 <contactref element="DRVMOT4_COM" pad="04"/>
-<contactref element="CAPTEUR1_COM" pad="01"/>
-<contactref element="CAPTEUR2_COM" pad="01"/>
-<contactref element="CAPTEUR3_COM" pad="01"/>
-<contactref element="CAPTEUR4_COM" pad="01"/>
 <contactref element="STOP_SENSOR1" pad="01"/>
 <contactref element="STOP_SENSOR2" pad="01"/>
@@
 <wire x1="16" y1="102" x2="16" y2="121.55" width="0.3048" layer="1"/>
 <wire x1="75" y1="107" x2="75" y2="84" width="0.3048" layer="1"/>
-<wire x1="55.52" y1="84" x2="40" y2="84" width="0.3048" layer="1"/>
-<wire x1="40" y1="84" x2="39.2" y2="84" width="0.3048" layer="1"/>
-<wire x1="39.2" y1="84" x2="39.2" y2="70.1825" width="0.3048" layer="1"/>
+<wire x1="55.52" y1="84" x2="34.12" y2="84" width="0.3048" layer="1"/>
 <wire x1="55.52" y1="84" x2="55.52" y2="64" width="0.3048" layer="1"/>
 <wire x1="55.52" y1="64" x2="55.52" y2="58.8825" width="0.3048" layer="1"/>
 <wire x1="75" y1="84" x2="55.52" y2="84" width="0.3048" layer="1"/>
-<wire x1="75" y1="84" x2="97.44" y2="84" width="0.3048" layer="1"/>
-<wire x1="97.44" y1="84" x2="97.44" y2="70.1825" width="0.3048" layer="1"/>
+<wire x1="75" y1="84" x2="92.36" y2="84" width="0.3048" layer="1"/>
+<wire x1="92.36" y1="84" x2="112.66" y2="84" width="0.3048" layer="1"/>
 <wire x1="5" y1="44.33" x2="5" y2="84" width="0.3048" layer="1"/>
-<wire x1="5" y1="84" x2="39.2" y2="84" width="0.3048" layer="1"/>
+<wire x1="5" y1="84" x2="34.12" y2="84" width="0.3048" layer="1"/>
 <wire x1="10.83" y1="44.33" x2="5" y2="44.33" width="0.3048" layer="1"/>
 <wire x1="5" y1="44.33" x2="5" y2="30" width="0.3048" layer="1"/>
 <wire x1="5" y1="30" x2="9.5" y2="30" width="0.3048" layer="1"/>
 <wire x1="9.5" y1="30" x2="9.5" y2="30.5475" width="0.3048" layer="1"/>
-<wire x1="112.66" y1="84" x2="97.44" y2="84" width="0.3048" layer="1"/>
 <wire x1="112.66" y1="84" x2="112.66" y2="61" width="0.3048" layer="1"/>
 <wire x1="112.66" y1="61" x2="112.66" y2="58.8825" width="0.3048" layer="1"/>
@@
 <wire x1="164.68" y1="84" x2="112.66" y2="84" width="0.3048" layer="16"/>
 <wire x1="164.68" y1="84" x2="164.68" y2="77" width="0.3048" layer="1"/>
-<wire x1="164.68" y1="77" x2="164.68" y2="70.1825" width="0.3048" layer="1"/>
 <wire x1="179.8" y1="77" x2="164.68" y2="77" width="0.3048" layer="1"/>
 <wire x1="179.8" y1="77" x2="179.8" y2="62" width="0.3048" layer="1"/>
@@
 <via x="112.66" y="84" extent="1-16" drill="0.8" diameter="1.27"/>
 <wire x1="234.34" y1="84" x2="234.34" y2="73" width="0.3048" layer="1"/>
-<wire x1="234.34" y1="73" x2="234.34" y2="70.1825" width="0.3048" layer="1"/>
 <via x="234.34" y="84" extent="1-16" drill="0.8" diameter="1.27"/>
 <wire x1="249.52" y1="73" x2="234.34" y2="73" width="0.3048" layer="1"/>
@@
 <wire x1="5" y1="84" x2="5" y2="91" width="0.3048" layer="1"/>
 <wire x1="5" y1="91" x2="16" y2="102" width="0.3048" layer="1"/>
+<contactref element="CAPTEUR4_COM" pad="03"/>
+<contactref element="CAPTEUR3_COM" pad="03"/>
+<contactref element="CAPTEUR2_COM" pad="03"/>
+<contactref element="CAPTEUR1_COM" pad="03"/>
+<wire x1="34.12" y1="84" x2="34.12" y2="70.1825" width="0.3048" layer="1"/>
+<wire x1="92.36" y1="84" x2="92.36" y2="70.1825" width="0.3048" layer="1"/>
+<wire x1="164.68" y1="77" x2="159.6" y2="77" width="0.3048" layer="1"/>
+<wire x1="159.6" y1="77" x2="159.6" y2="70.1825" width="0.3048" layer="1"/>
+<wire x1="234.34" y1="73" x2="229.26" y2="73" width="0.3048" layer="1"/>
+<wire x1="229.26" y1="73" x2="229.26" y2="70.1825" width="0.3048" layer="1"/>
 </signal>
 <signal name="MOTOR4_STEP">
@@
 </signal>
 </signals>
-<mfgpreviewcolors>
-<mfgpreviewcolor name="soldermaskcolor" color="0xC8008000"/>
-<mfgpreviewcolor name="silkscreencolor" color="0xFFFEFEFE"/>
-<mfgpreviewcolor name="backgroundcolor" color="0xFF282828"/>
-<mfgpreviewcolor name="coppercolor" color="0xFFFFBF00"/>
-<mfgpreviewcolor name="substratecolor" color="0xFF786E46"/>
-</mfgpreviewcolors>
+<errors>
+</errors>
 </board>
 </drawing>

Commit message: Add files via upload
Parts:
- C1, C2, C3, C4, C5: value 100uF -> 865060453008; device rcl:C1206K -> Condo-Wurth:CAP_865060453008_WRE
- moved C5 11.0 mm to (15.0, 55.0)
- moved C3 7.35 mm to (104.0, 29.0)
- moved C1 7.03 mm to (241.0, 30.0)
- moved C4 6.36 mm to (47.0, 29.0)
- moved C2 5.93 mm to (171.0, 30.0)
Routing:
- net MOT-: track 484.3 -> 604.7 mm
- net GND: track 1022.8 -> 980.7 mm, vias 19 -> 17
- net CAPTEUR_MOT4: track 29.3 -> 27.6 mm
- net CAPTEUR_MOT2: track 26.9 -> 25.4 mm
- net SUPPLY_COM: track 891.6 -> 892.4 mm

Commit message: Add files via upload
Routing:
- net MOT+: track 413.6 -> 409.6 mm
- net GND: track 980.7 -> 978.6 mm, vias 17 -> 16
- net SUPPLY_COM: track 892.4 -> 893.8 mm
