File: robot_vr.sch (EAGLE design)
At the start: 14 parts, among them CN10 SSM-119-L-DV, CN7 SSM-119-L-DV

Commit message: Add files via upload
Parts:
- removed DRIVER_MOT1, DRIVER_MOT2, DRIVER_MOT3, DRIVER_MOT4, DRIVER_MOT5: POLOLU-2134, POLOLU-2134:POLOLU-2134
- removed MOT5: 22-27-2041, 22-27-2041:22-27-2041
- added C2, C3, C4: 100uF, rcl:C-EUC1206K
- added CAPTEUR1_COM, CAPTEUR1_POW, CAPTEUR2_COM, CAPTEUR2_POW, CAPTEUR3_COM, CAPTEUR3_POW, CAPTEUR4_COM, CAPTEUR4_POW: SSM-103-S-SV, SSM-103-S-SV:SSM-103-S-SV
- added CAPTEUR_BUTEE: SSM-105-L-SV-BE, SSM-105-L-SV-BE:SSM-105-L-SV-BE
- added DRVMOT1_COM, DRVMOT1_POW, DRVMOT2_COM, DRVMOT2_POW, DRVMOT3_COM, DRVMOT3_POW, DRVMOT4_COM, DRVMOT4_POW: SSM-108-L-SV, SSM-108-L-SV:SSM-108-L-SV
Connections:
- removed net MOT1_ACTIVE: CN10.24, DRIVER_MOT1.STEP
- removed net MOT1_DIR: CN10.22, DRIVER_MOT1.DIR
- removed net MOT1_M0: CN10.30, DRIVER_MOT1.M0
- removed net MOT1_M1: CN10.28, DRIVER_MOT1.M1
- removed net MOT1_READY: CN10.26, DRIVER_MOT1.!SLP
- removed net MOT2_ACTIVE: CN10.31, DRIVER_MOT2.STEP
- removed net MOT2_DIR: CN10.33, DRIVER_MOT2.DIR
- removed net MOT2_M0: CN10.25, DRIVER_MOT2.M0
- removed net MOT2_M1: CN10.27, DRIVER_MOT2.M1
- removed net MOT2_READY: CN10.29, DRIVER_MOT2.!SLP
- removed net MOT3_ACTIVE: CN10.19, DRIVER_MOT3.STEP
- removed net MOT3_DIR: CN7.34, DRIVER_MOT3.DIR
- removed net MOT3_M0: CN10.13, DRIVER_MOT3.M0
- removed net MOT3_M1: CN10.15, DRIVER_MOT3.M1
- removed net MOT3_RADY: CN10.17
- removed net MOT3_READY: DRIVER_MOT3.!SLP
- removed net MOT4_ACTIVE: CN10.05, DRIVER_MOT4.STEP
- removed net MOT4_DIR: CN10.11, DRIVER_MOT4.DIR
- removed net MOT4_M0: CN7.36, DRIVER_MOT4.M0
- removed net MOT4_M1: CN10.01, DRIVER_MOT4.M1
- removed net MOT4_READY: CN10.03, DRIVER_MOT4.!SLP
- removed net MOT5_ACTIVE: CN7.23, DRIVER_MOT5.STEP
- removed net MOT5_DIR: CN7.35, DRIVER_MOT5.DIR
- removed net MOT5_M0: CN7.01, DRIVER_MOT5.M0
- removed net MOT5_M1: CN7.03, DRIVER_MOT5.M1
- removed net MOT5_READY: CN7.38, DRIVER_MOT5.!SLP
- removed net N$1: DRIVER_MOT1.A1, MOT1.1
- removed net N$10: ALIM_MOT-2.1, C1.2, DRIVER_MOT1.GND_MOT, DRIVER_MOT2.GND_MOT, DRIVER_MOT3.GND_MOT, DRIVER_MOT4.GND_MOT, DRIVER_MOT5.GND_MOT
- removed net N$11: DRIVER_MOT3.A1, MOT3.1
- removed net N$12: DRIVER_MOT3.A2, MOT3.2
- removed net N$13: DRIVER_MOT3.B1, MOT3.3
- removed net N$14: DRIVER_MOT3.B2, MOT3.4
- removed net N$15: DRIVER_MOT4.A1, MOT4.1
- removed net N$16: DRIVER_MOT4.A2, MOT4.2
- removed net N$17: DRIVER_MOT4.B1, MOT4.3
- removed net N$18: DRIVER_MOT4.B2, MOT4.4
- removed net N$19: DRIVER_MOT5.A1, MOT5.1
- removed net N$2: DRIVER_MOT1.A2, MOT1.2
- removed net N$20: DRIVER_MOT5.A2, MOT5.2
- removed net N$21: DRIVER_MOT5.B1, MOT5.3
- removed net N$22: DRIVER_MOT5.B2, MOT5.4
- removed net N$3: DRIVER_MOT1.B1, MOT1.3
- removed net N$4: DRIVER_MOT1.B2, MOT1.4
- removed net N$5: DRIVER_MOT2.A1, MOT2.1
- removed net N$6: DRIVER_MOT2.A2, MOT2.2
- removed net N$7: DRIVER_MOT2.B1, MOT2.3
- removed net N$8: DRIVER_MOT2.B2, MOT2.4
- removed net N$9: ALIM_MOT-1.1, C1.1, DRIVER_MOT1.VMOT, DRIVER_MOT2.VMOT, DRIVER_MOT3.VMOT, DRIVER_MOT4.VMOT, DRIVER_MOT5.VMOT
- new net BUTEE_M1: CAPTEUR_BUTEE.01, CN7.36
- new net BUTEE_M2: CAPTEUR_BUTEE.02, CN7.35
- new net BUTEE_M3: CAPTEUR_BUTEE.03, CN7.32
- new net BUTEE_M4: CAPTEUR_BUTEE.04, CN7.37
- new net BUTEE_M5: CAPTEUR_BUTEE.05, CN7.38
- new net CAPTEUR1: CAPTEUR1_COM.02
- new net CAPTEUR2: CAPTEUR2_COM.02
- new net CAPTEUR3: CAPTEUR3_COM.02
- new net CAPTEUR4: CAPTEUR4_COM.02
- new net CAPTEUR_MOT1: C1.1, CAPTEUR1_POW.03, DRVMOT1_POW.01
- new net CAPTEUR_MOT2: C2.1, CAPTEUR2_POW.03, DRVMOT2_POW.01
- new net CAPTEUR_MOT3: C3.1, CAPTEUR3_POW.03, DRVMOT3_POW.01
- new net CAPTEUR_MOT4: C4.1, CAPTEUR4_POW.03, DRVMOT4_POW.01
- new net CS: CN10.01
- new net MOSI: CN7.03
- new net MOT+: ALIM_MOT-1.1, CAPTEUR1_POW.01, CAPTEUR2_POW.01, CAPTEUR3_POW.01, CAPTEUR4_POW.01
- new net MOT-: ALIM_MOT-2.1, C1.2, C2.2, C3.2, C4.2, DRVMOT1_POW.02, DRVMOT2_POW.02, DRVMOT3_POW.02, DRVMOT4_POW.02
- new net MOT1_A1: DRVMOT1_POW.05, MOT1.3
- new net MOT1_A2: DRVMOT1_POW.06, MOT1.4
- new net MOT1_B1: DRVMOT1_POW.04, MOT1.2
- new net MOT1_B2: DRVMOT1_POW.03, MOT1.1
- new net MOT2_A1: DRVMOT2_POW.05, MOT2.3
- new net MOT2_A2: DRVMOT2_POW.06, MOT2.4
- new net MOT2_B1: DRVMOT2_POW.04, MOT2.2
- new net MOT2_B2: DRVMOT2_POW.03, MOT2.1
- new net MOT3_A1: DRVMOT3_POW.05, MOT3.3
- new net MOT3_A2: DRVMOT3_POW.06, MOT3.4
- new net MOT3_B1: DRVMOT3_POW.04, MOT3.2
- new net MOT3_B2: DRVMOT3_POW.03, MOT3.1
- new net MOT4_A1: DRVMOT4_POW.05, MOT4.3
- new net MOT4_A2: DRVMOT4_POW.06, MOT4.4
- new net MOT4_B1: DRVMOT4_POW.04, MOT4.2
- new net MOT4_B2: DRVMOT4_POW.03, MOT4.1
- new net MOT5_STEP: CN10.13
- new net MOTOR1_DIR: CN10.12, DRVMOT1_COM.08
- new net MOTOR1_READY: CN10.16, DRVMOT1_COM.06
- new net MOTOR1_STEP: CN10.14, DRVMOT1_COM.07
- new net MOTOR2_DIR: CN10.26, DRVMOT2_COM.08
- new net MOTOR2_READY: CN10.30, DRVMOT2_COM.06
- new net MOTOR2_STEP: CN10.28, DRVMOT2_COM.07
- new net MOTOR3_DIR: CN10.33, DRVMOT3_COM.08
- new net MOTOR3_READY: CN10.29, DRVMOT3_COM.06
- new net MOTOR3_STEP: CN10.31, DRVMOT3_COM.07
- new net MOTOR4_DIR: CN10.21, DRVMOT4_COM.08
- new net MOTOR4_READY: CN10.17, DRVMOT4_COM.06
- new net MOTOR4_STEP: CN10.19, DRVMOT4_COM.07
- new net MOTOR5_DIR: CN10.15
- new net MOTOR5_READY: CN10.11
- new net SCK/TX: CN7.01
- new net SCL: CN10.02
- new net SDA/MISO/RX: CN7.02
- new net SUPPLY_COM: CAPTEUR1_COM.01, CAPTEUR2_COM.01, CAPTEUR3_COM.01, CAPTEUR4_COM.01, CN7.06, DRVMOT1_COM.02, DRVMOT1_COM.03, DRVMOT1_COM.04, DRVMOT2_COM.02, DRVMOT2_COM.03, DRVMOT2_COM.04, DRVMOT3_COM.02, DRVMOT3_COM.03, DRVMOT3_COM.04, DRVMOT4_COM.02, DRVMOT4_COM.03, DRVMOT4_COM.04
- net GND: now also CAPTEUR1_COM.03, CAPTEUR2_COM.03, CAPTEUR3_COM.03, CAPTEUR4_COM.03, DRVMOT1_POW.08, DRVMOT2_POW.08, DRVMOT3_POW.08, DRVMOT4_POW.08; no longer DRIVER_MOT1.GND, DRIVER_MOT2.GND, DRIVER_MOT3.GND, DRIVER_MOT4.GND, DRIVER_MOT5.GND
Other:
- moved on the sheet: ALIM_MOT-1, ALIM_MOT-2, C1, MOT1, MOT2, MOT3, MOT4

Commit message: Add files via upload
Parts:
- added C5: 100uF, rcl:C-EUC1206K
- added MOTOR5_SERVO, STOP_SENSOR1, STOP_SENSOR2, STOP_SENSOR3, STOP_SENSOR4: SSM-103-S-SV, SSM-103-S-SV:SSM-103-S-SV
- added UART: 22-27-2041, 22-27-2041:22-27-2041
- renumbered CAPTEUR_BUTEE to CAM
Connections:
- removed net BUTEE_M1: CAM.01, CN7.36
- removed net BUTEE_M2: CAM.02, CN7.35
- removed net BUTEE_M3: CAM.03, CN7.32
- removed net BUTEE_M4: CAM.04, CN7.37
- removed net BUTEE_M5: CAM.05, CN7.38
- removed net CAPTEUR1: CAPTEUR1_COM.02
- removed net CAPTEUR2: CAPTEUR2_COM.02
- removed net CAPTEUR3: CAPTEUR3_COM.02
- removed net CAPTEUR4: CAPTEUR4_COM.02
- removed net MOT5_STEP: CN10.13
- removed net MOTOR5_DIR: CN10.15
- removed net MOTOR5_READY: CN10.11
- new net CURRENT_SENSOR1: CAPTEUR1_COM.02, CN7.28
- new net CURRENT_SENSOR2: CAPTEUR2_COM.02, CN7.30
- new net CURRENT_SENSOR3: CAPTEUR3_COM.02, CN7.34
- new net CURRENT_SENSOR4: CAPTEUR4_COM.02, CN7.36
- new net MOTOR5_SERVO: CN10.15, MOTOR5_SERVO.02
- new net STOP_SENSOR1: CN7.21, STOP_SENSOR1.02
- new net STOP_SENSOR2: CN7.23, STOP_SENSOR2.02
- new net STOP_SENSOR3: CN7.25, STOP_SENSOR3.02
- new net STOP_SENSOR4: CN7.27, STOP_SENSOR4.02
- new net UART1_RX: CN10.06, UART.2
- new net UART1_TX: CN10.34, UART.1
- new net UART2_RX: CN10.37, UART.4
- new net UART2_TX: CN10.35, UART.3
- net CS: now also CAM.01
- net GND: now also C5.2, MOTOR5_SERVO.03, STOP_SENSOR1.03, STOP_SENSOR2.03, STOP_SENSOR3.03, STOP_SENSOR4.03
- net MOSI: now also CAM.02
- net SCK/TX: now also CAM.04
- net SCL: now also CAM.05
- net SDA/MISO/RX: now also CAM.03
- net SUPPLY_COM: now also C5.1, MOTOR5_SERVO.01, STOP_SENSOR1.01, STOP_SENSOR2.01, STOP_SENSOR3.01, STOP_SENSOR4.01
Other:
- moved on the sheet: C1, C2, C3, C4, DRVMOT1_COM, DRVMOT1_POW, DRVMOT2_COM, DRVMOT2_POW, DRVMOT3_COM, DRVMOT3_POW, DRVMOT4_COM, DRVMOT4_POW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

Commit message: Add files via upload
Parts:
- removed UART: 22-27-2041, 22-27-2041:22-27-2041
Connections:
- removed net MOT+: ALIM_MOT-1.1, CAPTEUR1_POW.01, CAPTEUR2_POW.01, CAPTEUR3_POW.01, CAPTEUR4_POW.01
- removed net UART1_RX: CN10.06, UART.2
- removed net UART1_TX: CN10.34, UART.1
- removed net UART2_RX: CN10.37, UART.4
- removed net UART2_TX: CN10.35, UART.3
- new net N$1: ALIM_MOT-1.1, CAPTEUR1_POW.01, CAPTEUR2_POW.03, CAPTEUR3_POW.03, CAPTEUR4_POW.03
- net CAPTEUR_MOT2: now also CAPTEUR2_POW.01; no longer CAPTEUR2_POW.03
- net CAPTEUR_MOT3: now also CAPTEUR3_POW.01; no longer CAPTEUR3_POW.03
- net CAPTEUR_MOT4: now also CAPTEUR4_POW.01; no longer CAPTEUR4_POW.03
Other:
- moved on the sheet: ALIM_MOT-1, ALIM_MOT-2, C1, C2, C3, C4, C5, CAM, CAPTEUR1_COM, CAPTEUR1_POW, CAPTEUR2_COM, CAPTEUR2_POW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

Commit message: Add files via upload
Connections:
- net CS: now also CAM.04, CN10.02; no longer CAM.01, CN10.01
- net CURRENT_SENSOR1: now also CN7.27; no longer CN7.28
- net CURRENT_SENSOR2: now also CN7.29; no longer CN7.30
- net CURRENT_SENSOR3: now also CN7.33; no longer CN7.34
- net CURRENT_SENSOR4: now also CN7.35; no longer CN7.36
- net GND: now also CN7.07; no longer CN7.08
- net MOSI: now also CAM.01, CN7.04; no longer CAM.02, CN7.03
- net MOTOR1_DIR: now also CN10.11; no longer CN10.12
- net MOTOR1_READY: now also CN10.15; no longer CN10.16
- net MOTOR1_STEP: now also CN10.13; no longer CN10.14
- net MOTOR2_DIR: now also CN10.25; no longer CN10.26
- net MOTOR2_READY: now also CN10.29; no longer CN10.30
- net MOTOR2_STEP: now also CN10.27; no longer CN10.28
- net MOTOR3_DIR: now also CN10.34; no longer CN10.33
- net MOTOR3_READY: now also CN10.30; no longer CN10.29
- net MOTOR3_STEP: now also CN10.32; no longer CN10.31
- net MOTOR4_DIR: now also CN10.22; no longer CN10.21
- net MOTOR4_READY: now also CN10.18; no longer CN10.17
- net MOTOR4_STEP: now also CN10.20; no longer CN10.19
- net MOTOR5_SERVO: now also CN10.16; no longer CN10.15
- net SCK/TX: now also CAM.02, CN7.02; no longer CAM.04, CN7.01
- net SCL: now also CN10.01; no longer CN10.02
- net SDA/MISO/RX: now also CN7.01; no longer CN7.02
- net STOP_SENSOR1: now also CN7.22; no longer CN7.21
- net STOP_SENSOR2: now also CN7.24; no longer CN7.23
- net STOP_SENSOR3: now also CN7.26; no longer CN7.25
- net STOP_SENSOR4: now also CN7.28; no longer CN7.27
- net SUPPLY_COM: now also CN7.05; no longer CN7.06
Other:
- moved on the sheet: CN10

Commit message: Add files via upload
Connections:
- net N$1 renamed MOT+
Other:
- moved on the sheet: CN10, CN7

Commit message: Add files via upload
Connections:
- net CS: now also CAM.05; no longer CAM.04
- net MOSI: now also CAM.02; no longer CAM.01
- net SCK/TX: now also CAM.01; no longer CAM.02
- net SCL: now also CAM.04; no longer CAM.05
Changed lines of the file:
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@@
 <?xml version="1.0" encoding="utf-8"?>
 <!DOCTYPE eagle SYSTEM "eagle.dtd">
-<eagle version="7.6.0">
+<eagle version="9.6.2">
 <drawing>
 <settings>
 <setting alwaysvectorfont="no"/>
+<setting keepoldvectorfont="yes"/>
 <setting verticaltext="up"/>
 </settings>
@@
 <attribute name="VALUE" x="-132.715" y="-80.645" size="1.778" layer="96" rot="R180"/>
 </instance>
-<instance part="SUPPLY6" gate="GND" x="-35.56" y="50.8" rot="R90"/>
+<instance part="SUPPLY6" gate="GND" x="-35.56" y="50.8" smashed="yes" rot="R90">
+<attribute name="VALUE" x="-32.385" y="48.895" size="1.778" layer="96" rot="R90"/>
+</instance>
 </instances>
 <busses>
@@
 <net name="SCK/TX" class="0">
 <segment>
-<pinref part="CAM" gate="G$1" pin="02"/>
-<wire x1="137.16" y1="55.88" x2="124.46" y2="55.88" width="0.1524" layer="91"/>
-<label x="124.46" y="55.88" size="1.778" layer="95" rot="MR0"/>
-</segment>
-<segment>
 <pinref part="CN7" gate="G$1" pin="02"/>
 <wire x1="-63.5" y1="58.42" x2="-76.2" y2="58.42" width="0.1524" layer="91"/>
 <label x="-76.2" y="58.42" size="1.778" layer="95" rot="MR0"/>
 </segment>
+<segment>
+<pinref part="CAM" gate="G$1" pin="01"/>
+<wire x1="137.16" y1="58.42" x2="127" y2="58.42" width="0.1524" layer="91"/>
+<label x="127" y="58.42" size="1.778" layer="95" rot="R180"/>
+</segment>
 </net>
 <net name="MOSI" class="0">
-<segment>
-<pinref part="CAM" gate="G$1" pin="01"/>
-<wire x1="137.16" y1="58.42" x2="124.46" y2="58.42" width="0.1524" layer="91"/>
-<label x="124.46" y="58.42" size="1.778" layer="95" rot="MR0"/>
-</segment>
 <segment>
 <pinref part="CN7" gate="G$1" pin="04"/>
@@
 <label x="-76.2" y="55.88" size="1.778" layer="95" rot="MR0"/>
 </segment>
+<segment>
+<pinref part="CAM" gate="G$1" pin="02"/>
+<wire x1="137.16" y1="55.88" x2="127" y2="55.88" width="0.1524" layer="91"/>
+<label x="127" y="55.88" size="1.778" layer="95" rot="R180"/>
+</segment>
 </net>
 <net name="STOP_SENSOR4" class="0">
@@
 <net name="SDA/MISO/RX" class="0">
 <segment>
-<pinref part="CAM" gate="G$1" pin="03"/>
-<wire x1="137.16" y1="53.34" x2="127" y2="53.34" width="0.1524" layer="91"/>
-<label x="124.46" y="53.34" size="1.778" layer="95" rot="MR0"/>
-</segment>
-<segment>
 <pinref part="CN7" gate="G$1" pin="01"/>
 <wire x1="-38.1" y1="58.42" x2="-20.32" y2="58.42" width="0.1524" layer="91"/>
 <label x="-20.32" y="58.42" size="1.778" layer="95" rot="MR180"/>
 </segment>
+<segment>
+<pinref part="CAM" gate="G$1" pin="03"/>
+<wire x1="137.16" y1="53.34" x2="127" y2="53.34" width="0.1524" layer="91"/>
+<label x="127" y="53.34" size="1.778" layer="95" rot="R180"/>
+</segment>
 </net>
 <net name="STOP_SENSOR1" class="0">
@@
 <net name="CS" class="0">
 <segment>
-<pinref part="CAM" gate="G$1" pin="04"/>
-<wire x1="137.16" y1="50.8" x2="124.46" y2="50.8" width="0.1524" layer="91"/>
-<label x="124.46" y="50.8" size="1.778" layer="95" rot="MR0"/>
-</segment>
-<segment>
 <pinref part="CN10" gate="G$1" pin="02"/>
 <wire x1="43.18" y1="58.42" x2="30.48" y2="58.42" width="0.1524" layer="91"/>
 <label x="30.48" y="58.42" size="1.778" layer="95" rot="MR0"/>
 </segment>
+<segment>
+<pinref part="CAM" gate="G$1" pin="05"/>
+<wire x1="137.16" y1="48.26" x2="127" y2="48.26" width="0.1524" layer="91"/>
+<label x="127" y="48.26" size="1.778" layer="95" rot="R180"/>
+</segment>
 </net>
 <net name="MOTOR4_READY" class="0">
@@
 <net name="SCL" class="0">
 <segment>
-<pinref part="CAM" gate="G$1" pin="05"/>
-<wire x1="137.16" y1="48.26" x2="124.46" y2="48.26" width="0.1524" layer="91"/>
-<label x="124.46" y="48.26" size="1.778" layer="95" rot="MR0"/>
-</segment>
-<segment>
 <pinref part="CN10" gate="G$1" pin="01"/>
 <wire x1="68.58" y1="58.42" x2="83.82" y2="58.42" width="0.1524" layer="91"/>
 <label x="83.82" y="58.42" size="1.778" layer="95" rot="MR180"/>
+</segment>
+<segment>
+<pinref part="CAM" gate="G$1" pin="04"/>
+<wire x1="137.16" y1="50.8" x2="127" y2="50.8" width="0.1524" layer="91"/>
+<label x="127" y="50.8" size="1.778" layer="95" rot="R180"/>
 </segment>
 </net>
@@
 </sheet>
 </sheets>
-<errors>
-</errors>
 </schematic>
 </drawing>

Commit message: Add files via upload
Connections:
- net GND: now also CAPTEUR1_COM.01, CAPTEUR2_COM.01, CAPTEUR3_COM.01, CAPTEUR4_COM.01; no longer CAPTEUR1_COM.03, CAPTEUR2_COM.03, CAPTEUR3_COM.03, CAPTEUR4_COM.03
- net SUPPLY_COM: now also CAPTEUR1_COM.03, CAPTEUR2_COM.03, CAPTEUR3_COM.03, CAPTEUR4_COM.03; no longer CAPTEUR1_COM.01, CAPTEUR2_COM.01, CAPTEUR3_COM.01, CAPTEUR4_COM.01
Changed lines of the file:
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@@
 <?xml version="1.0" encoding="utf-8"?>
 <!DOCTYPE eagle SYSTEM "eagle.dtd">
-<eagle version="9.6.2">
+<eagle version="7.6.0">
 <drawing>
 <settings>
 <setting alwaysvectorfont="no"/>
-<setting keepoldvectorfont="yes"/>
 <setting verticaltext="up"/>
 </settings>
@@
 <part name="CN10" library="SSM-119-L-DV" deviceset="SSM-119-L-DV" device=""/>
 <part name="SUPPLY5" library="supply2" deviceset="GND" device=""/>
-<part name="SUPPLY7" library="supply2" deviceset="GND" device=""/>
-<part name="SUPPLY8" library="supply2" deviceset="GND" device=""/>
-<part name="SUPPLY9" library="supply2" deviceset="GND" device=""/>
-<part name="SUPPLY10" library="supply2" deviceset="GND" device=""/>
 <part name="C2" library="rcl" deviceset="C-EU" device="C1206K" value="100uF"/>
 <part name="MOT2" library="22-27-2041" deviceset="22-27-2041" device=""/>
@@
 <part name="SUPPLY14" library="supply2" deviceset="GND" device=""/>
 <part name="SUPPLY6" library="supply2" deviceset="GND" device=""/>
+<part name="SUPPLY15" library="supply2" deviceset="GND" device=""/>
+<part name="SUPPLY16" library="supply2" deviceset="GND" device=""/>
+<part name="SUPPLY17" library="supply2" deviceset="GND" device=""/>
+<part name="SUPPLY18" library="supply2" deviceset="GND" device=""/>
 </parts>
 <sheets>
@@
 <attribute name="VALUE" x="144.145" y="-114.935" size="1.778" layer="96" rot="MR0"/>
 </instance>
-<instance part="SUPPLY7" gate="GND" x="101.6" y="-50.8" smashed="yes" rot="R180">
-<attribute name="VALUE" x="103.505" y="-47.625" size="1.778" layer="96" rot="R180"/>
-</instance>
-<instance part="SUPPLY8" gate="GND" x="35.56" y="-50.8" smashed="yes" rot="R180">
-<attribute name="VALUE" x="37.465" y="-47.625" size="1.778" layer="96" rot="R180"/>
-</instance>
-<instance part="SUPPLY9" gate="GND" x="-33.02" y="-50.8" smashed="yes" rot="R180">
-<attribute name="VALUE" x="-31.115" y="-47.625" size="1.778" layer="96" rot="R180"/>
-</instance>
-<instance part="SUPPLY10" gate="GND" x="-101.6" y="-50.8" smashed="yes" rot="R180">
-<attribute name="VALUE" x="-99.695" y="-47.625" size="1.778" layer="96" rot="R180"/>
-</instance>
 <instance part="C2" gate="G$1" x="50.8" y="-114.3" smashed="yes" rot="MR0">
 <attribute name="NAME" x="49.276" y="-113.919" size="1.778" layer="95" rot="MR0"/>
@@
 <instance part="SUPPLY6" gate="GND" x="-35.56" y="50.8" smashed="yes" rot="R90">
 <attribute name="VALUE" x="-32.385" y="48.895" size="1.778" layer="96" rot="R90"/>
+</instance>
+<instance part="SUPPLY15" gate="GND" x="-96.52" y="-50.8" smashed="yes" rot="R180">
+<attribute name="VALUE" x="-94.615" y="-47.625" size="1.778" layer="96" rot="R180"/>
+</instance>
+<instance part="SUPPLY16" gate="GND" x="-27.94" y="-50.8" smashed="yes" rot="R180">
+<attribute name="VALUE" x="-26.035" y="-47.625" size="1.778" layer="96" rot="R180"/>
+</instance>
+<instance part="SUPPLY17" gate="GND" x="40.64" y="-50.8" smashed="yes" rot="R180">
+<attribute name="VALUE" x="42.545" y="-47.625" size="1.778" layer="96" rot="R180"/>
+</instance>
+<instance part="SUPPLY18" gate="GND" x="106.68" y="-50.8" smashed="yes" rot="R180">
+<attribute name="VALUE" x="108.585" y="-47.625" size="1.778" layer="96" rot="R180"/>
 </instance>
 </instances>
@@
 <nets>
 <net name="GND" class="0">
-<segment>
-<pinref part="SUPPLY7" gate="GND" pin="GND"/>
-<pinref part="CAPTEUR1_COM" gate="G$1" pin="03"/>
-</segment>
-<segment>
-<pinref part="SUPPLY8" gate="GND" pin="GND"/>
-<pinref part="CAPTEUR2_COM" gate="G$1" pin="03"/>
-</segment>
-<segment>
-<pinref part="SUPPLY9" gate="GND" pin="GND"/>
-<pinref part="CAPTEUR3_COM" gate="G$1" pin="03"/>
-</segment>
-<segment>
-<pinref part="SUPPLY10" gate="GND" pin="GND"/>
-<pinref part="CAPTEUR4_COM" gate="G$1" pin="03"/>
-</segment>
 <segment>
 <pinref part="SUPPLY5" gate="GND" pin="GND"/>
@@
 <pinref part="CN7" gate="G$1" pin="07"/>
 <pinref part="SUPPLY6" gate="GND" pin="GND"/>
+</segment>
+<segment>
+<pinref part="CAPTEUR4_COM" gate="G$1" pin="01"/>
+<pinref part="SUPPLY15" gate="GND" pin="GND"/>
+</segment>
+<segment>
+<pinref part="CAPTEUR3_COM" gate="G$1" pin="01"/>
+<pinref part="SUPPLY16" gate="GND" pin="GND"/>
+</segment>
+<segment>
+<pinref part="CAPTEUR2_COM" gate="G$1" pin="01"/>
+<pinref part="SUPPLY17" gate="GND" pin="GND"/>
+</segment>
+<segment>
+<pinref part="CAPTEUR1_COM" gate="G$1" pin="01"/>
+<pinref part="SUPPLY18" gate="GND" pin="GND"/>
 </segment>
 </net>
@@
 </segment>
 <segment>
-<wire x1="106.68" y1="-53.34" x2="106.68" y2="-38.1" width="0.1524" layer="91"/>
-<label x="106.68" y="-38.1" size="1.778" layer="95" rot="R90"/>
-<pinref part="CAPTEUR1_COM" gate="G$1" pin="01"/>
-</segment>
-<segment>
-<wire x1="40.64" y1="-53.34" x2="40.64" y2="-38.1" width="0.1524" layer="91"/>
-<label x="40.64" y="-38.1" size="1.778" layer="95" rot="R90"/>
-<pinref part="CAPTEUR2_COM" gate="G$1" pin="01"/>
-</segment>
-<segment>
-<wire x1="-27.94" y1="-53.34" x2="-27.94" y2="-38.1" width="0.1524" layer="91"/>
-<label x="-27.94" y="-38.1" size="1.778" layer="95" rot="R90"/>
-<pinref part="CAPTEUR3_COM" gate="G$1" pin="01"/>
-</segment>
-<segment>
-<wire x1="-96.52" y1="-53.34" x2="-96.52" y2="-38.1" width="0.1524" layer="91"/>
-<label x="-96.52" y="-38.1" size="1.778" layer="95" rot="R90"/>
-<pinref part="CAPTEUR4_COM" gate="G$1" pin="01"/>
-</segment>
-<segment>
 <pinref part="STOP_SENSOR1" gate="G$1" pin="01"/>
 <wire x1="-139.7" y1="58.42" x2="-127" y2="58.42" width="0.1524" layer="91"/>
@@
 <wire x1="-38.1" y1="53.34" x2="-20.32" y2="53.34" width="0.1524" layer="91"/>
 <label x="-20.32" y="53.34" size="1.778" layer="95"/>
+</segment>
+<segment>
+<pinref part="CAPTEUR4_COM" gate="G$1" pin="03"/>
+<wire x1="-101.6" y1="-53.34" x2="-101.6" y2="-38.1" width="0.1524" layer="91"/>
+<label x="-101.6" y="-38.1" size="1.778" layer="95" rot="R90"/>
+</segment>
+<segment>
+<pinref part="CAPTEUR3_COM" gate="G$1" pin="03"/>
+<wire x1="-33.02" y1="-53.34" x2="-33.02" y2="-38.1" width="0.1524" layer="91"/>
+<label x="-33.02" y="-38.1" size="1.778" layer="95" rot="R90"/>
+</segment>
+<segment>
+<pinref part="CAPTEUR2_COM" gate="G$1" pin="03"/>
+<wire x1="35.56" y1="-53.34" x2="35.56" y2="-38.1" width="0.1524" layer="91"/>
+<label x="35.56" y="-38.1" size="1.778" layer="95" rot="R90"/>
+</segment>
+<segment>
+<pinref part="CAPTEUR1_COM" gate="G$1" pin="03"/>
+<wire x1="101.6" y1="-53.34" x2="101.6" y2="-38.1" width="0.1524" layer="91"/>
+<label x="101.6" y="-38.1" size="1.778" layer="95" rot="R90"/>
 </segment>
 </net>
@@
 </sheet>
 </sheets>
+<errors>
+</errors>
 </schematic>
 </drawing>

Commit message: Add files via upload
Parts:
- C1, C2, C3, C4, C5: value 100uF -> 865060453008; device rcl:C-EUC1206K -> Condo-Wurth:865060453008
